File: eagle/controller/controller.sch (EAGLE design)
At the start: 11 parts, among them Q1 FQP30N06L, SW1 Select, U1 HI4030, U2 DS18B20, U3 ARDUINO_PRO_MICRO

Commit message: bom: Updated bill of materials. eagle: Updated controller.sch and controller.pdf. howto: Added controller.pdf.
Other:
- note added: "Two DS18B20 are required."
Changed lines of the file:
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@@
  PARTICULAR PURPOSE. Please see the CERN OHL v.1.2 for applicable
  conditions</text>
+<text x="25.4" y="121.92" size="1.778" layer="97">Two DS18B20 are required.</text>
 </plain>
 <instances>
